File: 24v-logic.kicad_sch (KiCad schematic)
At the start: 55 parts

Commit message: Changes for missing components and migrating to KiCAD 6
Parts:
- removed D1, D2, D3, D4, D5, D6, D7, D8: (no value), symbol Device:D_Zener
- removed D10, D11, D12, D13, D14, D15, D16, D9: (no value), symbol Device:D
- removed D17, D18, D19, D20, D21, D22, D23, D24: (no value), symbol Device:LED
- removed R1, R10, R11, R12, R13, R14, R15, R16, R17, R18, R19, R2, R20, R21, R22, R23, R24, R3, R4, R5, R6, R7, R8, R9: (no value), symbol Device:R
- H1, H2, H3, H4: value (none) -> MountingHole; footprint (none) -> MountingHole:MountingHole_3.2mm_M3; now left out of the parts list
- J1, J3: value (none) -> Conn_02x10_Odd_Even; footprint (none) -> Connector_IDC:IDC-Header_2x10_P2.54mm_Vertical; now left out of the parts list
- J2: value (none) -> Screw_Terminal_01x09; footprint (none) -> Connector_Phoenix_MC:PhoenixContact_MCV_1,5_9-G-3.81_1x09_P3.81mm_Vertical; now left out of the parts list
Other:
- added sheet Voltage Divider (voltage-divider.kicad_sch)
- added sheet Voltage Divider1 (voltage-divider.kicad_sch)
- added sheet Voltage Divider2 (voltage-divider.kicad_sch)
- added sheet Voltage Divider3 (voltage-divider.kicad_sch)
- added sheet Voltage Divider4 (voltage-divider.kicad_sch)
- added sheet Voltage Divider5 (voltage-divider.kicad_sch)
- added sheet Voltage Divider6 (voltage-divider.kicad_sch)
- added sheet Voltage Divider7 (voltage-divider.kicad_sch)
